File: 07_LBAM_DFR.kicad_pcb (KiCad board)
At the start: 2 copper layers, 100 x 80 mm, 23 parts, among them J1 Conn_01x01, J18 Conn_01x02, J2 Conn_01x01, J26 Conn_01x02, J27 Conn_01x02, J3 Conn_01x01, J4 Conn_01x02, J5 Conn_01x02, J9 Conn_01x02, Q1 2N7002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

Commit message: maj split librairies
Parts:
- U1: footprint Chimere:MODULE_DFR0299 -> Chimere_comps:MODULE_DFR0299
- U2: footprint Chimere:MODULE_ESP32-DEVKITC -> Chimere_comps:MODULE_ESP32-DEVKITC
- U4: footprint Chimere:Batt_Alim -> Chimere_mods:Batt_Alim
