File: Batt_alim.sch (KiCad schematic (older format))
At the start: 4 parts, among them J27 Conn_01x02, J4 Conn_01x02, J9 Conn_01x02, U4 Batt_Alim

Commit message: maj split librairies
Parts:
- U4: footprint Chimere:Batt_Alim -> Chimere_mods:Batt_Alim; symbol Chimere:Batt_Alim -> Chimere_mods:Batt_Alim
Changed lines of the file:
@@
 $EndDescr
 $Comp
-L Chimere:Batt_Alim U4
+L Chimere_mods:Batt_Alim U4
 U 1 1 5FDF7692
 P 6300 3750
+AR Path="/5FDF7692" Ref="U4"  Part="1"
+AR Path="/5FC6D1FC/5FDF7692" Ref="U4"  Part="1"
 F 0 "U4" H 6300 4290 50  0000 C CNN
 F 1 "Batt_Alim" H 6300 4199 50  0000 C CNN
-F 2 "Chimere:Batt_Alim" H 6300 3750 50  0001 C CNN
+F 2 "Chimere_mods:Batt_Alim" H 6300 3750 50  0001 C CNN
 F 3 "" H 6300 3750 50  0001 C CNN
 	1    6300 3750
