File: audio.sch (KiCad schematic (older format))
At the start: 5 parts, among them J1 Conn_01x01, J2 Conn_01x01, J3 Conn_01x01, J5 Conn_01x02, U1 DFR0299

Commit message: maj split librairies
Parts:
- U1: footprint Chimere:MODULE_DFR0299 -> Chimere_comps:MODULE_DFR0299; symbol Chimere:DFR0299 -> Chimere_comps:DFR0299
Changed lines of the file:
@@
 $EndDescr
 $Comp
-L Chimere:DFR0299 U1
+L Chimere_comps:DFR0299 U1
 U 1 1 5FC6C86F
 P 6125 2350
+AR Path="/5FC6C86F" Ref="U1"  Part="1"
+AR Path="/5FC6C772/5FC6C86F" Ref="U1"  Part="1"
 F 0 "U1" H 6125 3217 50  0000 C CNN
 F 1 "DFR0299" H 6125 3126 50  0000 C CNN
-F 2 "Chimere:MODULE_DFR0299" H 6125 2350 50  0001 L BNN
+F 2 "Chimere_comps:MODULE_DFR0299" H 6125 2350 50  0001 L BNN
 F 3 "" H 6125 2350 50  0001 L BNN
 F 4 "Dfplayer - a Mini Mp3 Player" H 6125 2350 50  0001 L BNN "DESCRIPTION"
