File: esp32.sch (KiCad schematic (older format))
At the start: 12 parts, among them J18 Conn_01x02, J26 Conn_01x02, Q1 2N7002, U2 ESP32-DEVKITC

Commit message: maj split librairies
Parts:
- U2: footprint Chimere:MODULE_ESP32-DEVKITC -> Chimere_comps:MODULE_ESP32-DEVKITC; symbol Chimere:ESP32-DEVKITC -> Chimere_comps:ESP32-DEVKITC
Changed lines of the file:
@@
 $EndDescr
 $Comp
-L Chimere:ESP32-DEVKITC U2
+L Chimere_comps:ESP32-DEVKITC U2
 U 1 1 5FC6D4F6
 P 6900 3525
+AR Path="/5FC6D4F6" Ref="U2"  Part="1"
+AR Path="/5FC6D1B4/5FC6D4F6" Ref="U2"  Part="1"
 F 0 "U2" H 6900 4692 50  0000 C CNN
 F 1 "ESP32-DEVKITC" H 6900 4601 50  0000 C CNN
-F 2 "Chimere:MODULE_ESP32-DEVKITC" H 6900 3525 50  0001 L BNN
+F 2 "Chimere_comps:MODULE_ESP32-DEVKITC" H 6900 3525 50  0001 L BNN
 F 3 "" H 6900 3525 50  0001 L BNN
 F 4 "Manufacturer Recommendations" H 6900 3525 50  0001 L BNN "STANDARD"
